Commit message: remove eef

File: kr210_pen_support/urdf/kr210_pen.urdf (robot description, URDF)
Before this commit: robot kr210_pen, 17 links, 16 joints
Links:
- removed link penholder_base_link
- removed link penholder_tool_tip
- added link kr210_qr_tool0
- added link quickrelease_base_link; collision mesh filename=package://kr210_robot_support/meshes/collision/KUKA_Quickre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 scale=0.001 0.001 0.001; visual mesh filename=package://kr210_robot_support/meshes/visual/KUKA_Quickrelea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 scale=0.001 0.001 0.001
Joints:
- removed joint penholder_base_link_to_kr210_tool0
- removed joint penholder_tool_tip_to_penholder_base_link
- removed joint table_base_link_to_kl2000_mobile_base
- added joint base_link_to_kl2000_mobile_base: type fixed, parent kl2000_base_link, child table_base_link, origin xyz=-1.264 1.719 0.3475 rpy=0 0 -1.57079632679
- added joint kr210_tool0_to_{prefix}quickrelease_base_link: type fixed, parent kr210_tool0, child quickrelease_base_link, origin xyz=0 0 0 rpy=1.57079632679 0 0
- added joint tool0_to_quickrelease_base: type fixed, parent quickrelease_base_link, child kr210_qr_tool0, origin xyz=0 0.05 0 rpy=-1.57079632679 0 0

File: kr210_pen_support/urdf/macros/kr210_pen_macro.xacro (robot description, xacro)
@@ -11,9 +11,7 @@
   <xacro:include filename="$(find kr210_pen_support)/urdf/parts/kl2000_console_h400_macro.xacro"/>
   <!-- Kuka KR210R2700extra robot -->
-  <xacro:include filename="$(find kuka_kr210_support)/urdf/kr210r2700extra_macro.xacro"/>
+  <xacro:include filename="$(find kr210_robot_support)/urdf/macros/kr210_macro.xacro"/>
   <!-- Welding Table -->
   <xacro:include filename="$(find kr210_pen_support)/urdf/parts/forster_welding_table_macro.xacro"/>
-  <!-- Penholder End Effector -->
-  <xacro:include filename="$(find kr210_eef_support)/urdf/penholder_macro.xacro"/>
   <!-- MACRO START  -->
   <xacro:macro name="kr210_pen" params="prefix">
@@ -21,7 +19,6 @@
     <xacro:kl2000 prefix="${prefix}kl2000_"/>
     <xacro:kl2000_console_h400 prefix="${prefix}console_"/>
-    <xacro:kuka_kr210r2700extra prefix="${prefix}kr210_"/>
+    <xacro:kr210 prefix="${prefix}"/>
     <xacro:forster_welding_table prefix="${prefix}table_"/>
-    <xacro:penholder prefix="${prefix}penholder_"/>
     <!-- JOINTS -->
     <!-- Console to Linear track -->
@@ -38,15 +35,9 @@
     </joint>
     <!-- Welding table to linear track -->
-    <joint name="${prefix}table_base_link_to_${prefix}kl2000_mobile_base" type="fixed">
+    <joint name="${prefix}base_link_to_${prefix}kl2000_mobile_base" type="fixed">
       <parent link="${prefix}kl2000_base_link"/>
       <child link="${prefix}table_base_link"/>
       <origin xyz="-1.264 1.719 ${(table_height - table_top_thickness)/2}" rpy="0 0 ${-pi/2}"/>
     </joint>
-    <!-- End effector to robot -->
-    <joint name="${prefix}penholder_base_link_to_${prefix}kr210_tool0" type="fixed">
-      <parent link="${prefix}kr210_tool0"/>
-      <child link="${prefix}penholder_base_link"/>
-      <origin xyz="0 0 0" rpy="0 0 0"/>
-    </joint>
   </xacro:macro>
 </robot>

File: kr210_pen_support/urdf/parts/kl2000_console_h400_macro.xacro (robot description, xacro)
@@ -6,5 +6,5 @@
         <origin xyz="0 0 0" rpy="0 0 0"/>
         <geometry>
-          <mesh filename="package://kr210_pen_support/meshes/visual/kl2000_console_h400.dae"/>
+          <mesh filename="package://kr210_pen_support/meshes/visual/kl2000_console_h400.dae" />
         </geometry>
       </visual>
@@ -12,5 +12,5 @@
         <origin xyz="0 0 0" rpy="0 0 0"/>
         <geometry>
-          <mesh filename="package://kr210_pen_support/meshes/collision/kl2000_console_h400_collision.stl"/>
+          <mesh filename="package://kr210_pen_support/meshes/collision/kl2000_console_h400_collision.stl" />
         </geometry>
       </collision>
