Commit message: Delete error related with micros folder incorrect naming

File: kr210_pen_support/urdf/macros/kr210_pen_macro.xacro (robot description, xacro)
@@ -15,10 +15,9 @@
   <xacro:include filename="$(find kr210_pen_support)/urdf/parts/forster_welding_table_macro.xacro"/>
   <!-- MACRO START  -->
-  <xacro:macro name="kr210_no_eef_cell" params="prefix">
+  <xacro:macro name="kr210_pen" params="prefix">
     <!-- DEFINITIONS -->
     <xacro:kl2000 prefix="${prefix}kl2000_"/>
     <xacro:kl2000_console_h400 prefix="${prefix}console_"/>
     <xacro:kr210 prefix="${prefix}"/>
-    <xacro:kr1_hc1000_r1280 prefix="${prefix}kr1_"/>
     <xacro:forster_welding_table prefix="${prefix}table_"/>
     <!-- JOINTS -->
@@ -39,5 +38,5 @@
       <parent link="${prefix}kl2000_base_link"/>
       <child link="${prefix}table_base_link"/>
-      <origin xyz="1.264 0.919 ${(table_height - table_top_thickness)/2}" rpy="0 0 0"/>
+      <origin xyz="-1.264 1.419 ${(table_height - table_top_thickness)/2}" rpy="0 0 ${-pi/2}"/>
     </joint>
   </xacro:macro>

File: kr210_pen_support/urdf/parts/forster_welding_table_macro.xacro (robot description, xacro)
@@ -4,49 +4,49 @@
   <xacro:include filename="$(find kuka_resources)/urdf/common_materials.xacro"/>
   <!-- Defining variables -->
-	<!-- min:410 mm max:1200 mm Forster HW4002-->
-  <xacro:property name="table_height" value="0.78"/>
-  <xacro:property name="table_width" value="1.2"/>
-  <xacro:property name="table_length" value="2.5"/>
-  <xacro:property name="table_top_thickness" value="0.085"/>
-  <xacro:property name="table_top_overhang" value="0.2"/>
-	<xacro:macro name="forster_welding_table" params="prefix">
-		<!-- LINK DEFINITIONS -->
-		<link name="${prefix}base_link">
-			<visual>
-				<origin xyz="0 0 0" rpy="0 0 0"/>
-					<geometry>
-						<box size ="${table_width-table_top_overhang} ${table_length-table_top_overhang} ${table_height - table_top_thickness}"/>
-					</geometry>
-          <material name="">
-            <color rgba="${colour_kuka_anthracite_gray}"/>
-          </material>
-			</visual>
-			<collision>
-				<origin xyz="0 0 0" rpy="0 0 0"/>
-					<geometry>
-						<box size="${table_width-table_top_overhang} ${table_length-table_top_overhang} ${table_height - table_top_thickness}"/>
-					</geometry>
-			</collision>
-		</link>
+  <!-- min:410 mm max:1200 mm Forster HW4002-->
+  <xacro:property name="table_height" value="0.78"/> <!--0.78-->
+  <xacro:property name="table_width" value="1.2"/> <!--1.2-->
+  <xacro:property name="table_length" value="2.5"/> <!--2.5-->
+  <xacro:property name="table_top_thickness" value="0.085"/> <!--0.085-->
+  <xacro:property name="table_top_overhang" value="0.2"/> <!--0.2-->
+  <xacro:macro name="forster_welding_table" params="prefix">
+    <!-- LINK DEFINITIONS -->
+    <link name="${prefix}base_link">
+      <visual>
+        <origin xyz="0 0 0" rpy="0 0 0"/>
+        <geometry>
+          <box size ="${table_width-table_top_overhang} ${table_length-table_top_overhang} ${table_height - table_top_thickness}"/>
+        </geometry>
+        <material name="">
+          <color rgba="${colour_kuka_anthracite_gray}"/>
+        </material>
+      </visual>
+      <collision>
+        <origin xyz="0 0 0" rpy="0 0 0"/>
+        <geometry>
+          <box size="${table_width-table_top_overhang} ${table_length-table_top_overhang} ${table_height - table_top_thickness}"/>
+        </geometry>
+      </collision>
+    </link>
     <!-- Geometry model table top -->
     <link name="${prefix}table_top">
-    <visual>
+      <visual>
         <origin xyz="${table_length/2} ${-table_top_thickness/2} ${table_width/2}" rpy="0 0 0"/>
-          <geometry>
-            <box size ="${table_length} ${-table_top_thickness} ${table_width}"/>
-          </geometry>
-          <material name="">
-            <color rgba="${colour_kuka_anthracite_gray}"/>
-          </material>
+        <geometry>
+          <box size ="${table_length} ${-table_top_thickness} ${table_width}"/>
+        </geometry>
+        <material name="">
+          <color rgba="${colour_kuka_anthracite_gray}"/>
+        </material>
       </visual>
       <collision>
         <origin xyz="${table_length/2} ${-table_top_thickness/2} ${table_width/2}" rpy="0 0 0"/>
         <geometry>
-            <box size ="${table_length} ${table_top_thickness} ${table_width}"/>
+          <box size ="${table_length} ${table_top_thickness} ${table_width}"/>
         </geometry>
       </collision>
     </link>
-<!-- CAD model table top -->
-<!-- 		<link name="${prefix}table_top">
+    <!-- CAD model table top -->
+    <!-- 		<link name="${prefix}table_top">
       <visual>
       	<origin xyz="0 0 0" rpy="0 0 0"/>
@@ -62,5 +62,5 @@
       </collision>
     </link> -->
-		 <!-- JOINT DEFINITIONS -->
+    <!-- JOINT DEFINITIONS -->
     <joint name="${prefix}base_link_joint" type="fixed">
       <origin xyz="${-table_width/2} ${-table_length/2} ${(table_height/2) + (table_top_thickness/2)}" rpy="${pi/2} 0 ${pi/2}"/>
@@ -68,4 +68,4 @@
       <child link="${prefix}table_top"/>
     </joint>
-		</xacro:macro>
+  </xacro:macro>
 </robot>

Commit message: Add moveit configuration folder

File: kr210_pen_support/urdf/macros/kr210_pen_macro.xacro (robot description, xacro)
@@ -38,5 +38,5 @@
       <parent link="${prefix}kl2000_base_link"/>
       <child link="${prefix}table_base_link"/>
-      <origin xyz="-1.264 1.419 ${(table_height - table_top_thickness)/2}" rpy="0 0 ${-pi/2}"/>
+      <origin xyz="-1.264 1.719 ${(table_height - table_top_thickness)/2}" rpy="0 0 ${-pi/2}"/>
     </joint>
   </xacro:macro>

Commit message: Add eef

File: kr210_pen_support/urdf/macros/kr210_pen_macro.xacro (robot description, xacro)
@@ -14,4 +14,6 @@
   <!-- Welding Table -->
   <xacro:include filename="$(find kr210_pen_support)/urdf/parts/forster_welding_table_macro.xacro"/>
+  <!-- Penholder End Effector -->
+  <xacro:include filename="$(find kr210_pen_support)/urdf/parts/penholder_macro.xacro"/>
   <!-- MACRO START  -->
   <xacro:macro name="kr210_pen" params="prefix">
@@ -21,4 +23,5 @@
     <xacro:kr210 prefix="${prefix}"/>
     <xacro:forster_welding_table prefix="${prefix}table_"/>
+    <xacro:penholder prefix="${prefix}penholder_"/>
     <!-- JOINTS -->
     <!-- Console to Linear track -->
@@ -40,4 +43,10 @@
       <origin xyz="-1.264 1.719 ${(table_height - table_top_thickness)/2}" rpy="0 0 ${-pi/2}"/>
     </joint>
+    <!-- End effector to robot -->
+    <joint name="${prefix}penholder_eef_base_link_to_${prefix}quick_release_base_link" type="fixed">
+      <parent link="${prefix}kr210_qr_tool0"/>
+      <child link="${prefix}penholder_base_link"/>
+      <origin xyz="0 0 0.02" rpy="${pi} 0 ${pi*(5/6)}"/>
+    </joint>
   </xacro:macro>
 </robot>

File: kr210_pen_support/urdf/parts/kl2000_console_h400_macro.xacro (robot description, xacro)
@@ -6,5 +6,5 @@
         <origin xyz="0 0 0" rpy="0 0 0"/>
         <geometry>
-          <mesh filename="package://kr210_pen_support/meshes/visual/kl2000_console_h400.dae" />
+          <mesh filename="package://kr210_pen_support/meshes/visual/kl2000_console_h400.dae"/>
         </geometry>
       </visual>
@@ -12,5 +12,5 @@
         <origin xyz="0 0 0" rpy="0 0 0"/>
         <geometry>
-          <mesh filename="package://kr210_pen_support/meshes/collision/kl2000_console_h400_collision.stl" />
+          <mesh filename="package://kr210_pen_support/meshes/collision/kl2000_console_h400_collision.stl"/>
         </geometry>
       </collision>

Commit message: rotate table

File: kr210_pen_support/urdf/macros/kr210_pen_macro.xacro (robot description, xacro)
@@ -38,5 +38,5 @@
       <parent link="${prefix}kl2000_base_link"/>
       <child link="${prefix}table_base_link"/>
-      <origin xyz="-1.264 1.719 ${(table_height - table_top_thickness)/2}" rpy="0 0 ${-pi/2}"/>
+      <origin xyz="-1.264 1.719 ${(table_height - table_top_thickness)/2}" rpy="0 0 ${pi/2}"/>
     </joint>
   </xacro:macro>

Commit message: add rsi files

File: kr210_pen_support/urdf/macros/kr210_pen_macro.xacro (robot description, xacro)
@@ -41,5 +41,6 @@
       <parent link="${prefix}kl2000_base_link"/>
       <child link="${prefix}table_base_link"/>
-      <origin xyz="-1.264 1.719 ${(table_height - table_top_thickness)/2}" rpy="0 0 ${-pi/2}"/>
+     <origin xyz="-1.264 1.719 ${(table_height - table_top_thickness)/2}" rpy="0 0 ${-pi/2}"/>
+      <!-- <origin xyz="1.264 0.919 ${(table_height - table_top_thickness)/2}" rpy="0 0 0"/>   -->
     </joint>
     <!-- End effector to robot -->

Commit message: add kuka drivers and change position of the table

File: kr210_pen_support/urdf/macros/kr210_pen_macro.xacro (robot description, xacro)
@@ -41,6 +41,6 @@
       <parent link="${prefix}kl2000_base_link"/>
       <child link="${prefix}table_base_link"/>
-     <origin xyz="-1.264 1.719 ${(table_height - table_top_thickness)/2}" rpy="0 0 ${-pi/2}"/>
-      <!-- <origin xyz="1.264 0.919 ${(table_height - table_top_thickness)/2}" rpy="0 0 0"/>   -->
+     <!-- <origin xyz="-1.264 1.719 ${(table_height - table_top_thickness)/2}" rpy="0 0 ${-pi/2}"/>        -->
+      <origin xyz="1.264 0.919 ${(table_height - table_top_thickness)/2}" rpy="0 0 0"/>
     </joint>
     <!-- End effector to robot -->

Commit message: remove table from urdf and srdf

File: kr210_pen_support/urdf/macros/kr210_pen_macro.xacro (robot description, xacro)
@@ -13,5 +13,5 @@
   <xacro:include filename="$(find kuka_kr210_support)/urdf/kr210r2700extra_macro.xacro"/>
   <!-- Welding Table -->
-  <xacro:include filename="$(find kr210_pen_support)/urdf/parts/forster_welding_table_macro.xacro"/>
+  <!-- <xacro:include filename="$(find kr210_pen_support)/urdf/parts/forster_welding_table_macro.xacro"/> -->
   <!-- Penholder End Effector -->
   <xacro:include filename="$(find kr210_eef_support)/urdf/penholder_macro.xacro"/>
@@ -22,5 +22,5 @@
     <xacro:kl2000_console_h400 prefix="${prefix}console_"/>
     <xacro:kuka_kr210r2700extra prefix="${prefix}kr210_"/>
-    <xacro:forster_welding_table prefix="${prefix}table_"/>
+    <!-- <xacro:forster_welding_table prefix="${prefix}table_"/> -->
     <xacro:penholder prefix="${prefix}penholder_"/>
     <!-- JOINTS -->
@@ -38,10 +38,9 @@
     </joint>
     <!-- Welding table to linear track -->
-    <joint name="${prefix}table_base_link_to_${prefix}kl2000_mobile_base" type="fixed">
+    <!-- <joint name="${prefix}table_base_link_to_${prefix}kl2000_mobile_base" type="fixed">
       <parent link="${prefix}kl2000_base_link"/>
       <child link="${prefix}table_base_link"/>
      <origin xyz="-1.264 1.719 ${(table_height - table_top_thickness)/2}" rpy="0 0 ${-pi/2}"/>
-      <!-- <origin xyz="1.264 0.919 ${(table_height - table_top_thickness)/2}" rpy="0 0 0"/>   -->
-    </joint>
+    </joint> -->
     <!-- End effector to robot -->
     <joint name="${prefix}penholder_base_link_to_${prefix}kr210_tool0" type="fixed">
