Commit message: Remove a minus in one of the size of the table

File: kr210_pen_support/urdf/parts/forster_welding_table_macro.xacro (robot description, xacro)
@@ -34,5 +34,5 @@
         <origin xyz="${table_length/2} ${-table_top_thickness/2} ${table_width/2}" rpy="0 0 0"/>
         <geometry>
-          <box size ="${table_length} ${-table_top_thickness} ${table_width}"/>
+          <box size ="${table_length} ${table_top_thickness} ${table_width}"/>
         </geometry>
         <material name="">
