Commit message: Pen end-effector in correct position

File: kr210_eef_support/urdf/penholder_macro.xacro (robot description, xacro)
@@ -1,4 +1,6 @@
 <?xml version="1.0"?>
 <robot xmlns:xacro="http://wiki.ros.org/xacro">
+  <xacro:property name="eef_bottom_distance_from_center" value="0.1898"/>
+  <xacro:property name="eef_tip_distance_from_center" value="0.2294"/>
     <xacro:macro name="penholder" params="prefix">
         <!--<link name="${prefix}base_link">
@@ -18,21 +20,26 @@
         <link name="${prefix}base_link">
             <visual>
-                <origin xyz="0 0 -0.2" rpy="${pi/2} 0 0"/>
+                <origin xyz="0 0 ${eef_bottom_distance_from_center}" rpy="${-pi/2} 0 0"/>
                 <geometry>
-                    <mesh filename="package://kr210_pen_support/meshes/visual/penholder.dae" scale="0.001 0.001 0.001"/>
+                    <mesh filename="package://kr210_eef_support/meshes/visual/penholder.dae" scale="0.001 0.001 0.001"/>
                 </geometry>
             </visual>
             <collision>
-                <origin xyz="0 0 -0.2" rpy="${pi/2} 0 0"/>
+                <origin xyz="0 0 ${eef_bottom_distance_from_center}" rpy="${-pi/2} 0 0"/>
                 <geometry>
-                    <mesh filename="package://kr210_pen_support/meshes/collision/penholder.stl" scale="0.001 0.001 0.001"/>
+                    <mesh filename="package://kr210_eef_support/meshes/collision/penholder.stl" scale="0.001 0.001 0.001"/>
                 </geometry>
             </collision>
         </link>
         <link name="${prefix}tool_tip"/>
-        <joint name="${prefix}eef_base_link_to_${prefix}base_link" type="fixed">
+        <!-- <joint name="${prefix}eef_base_link_to_${prefix}base_link" type="fixed">
+            <parent link= "${prefix}base_link"/>
+            <child link= "${prefix}eef_base_link"/>
+            <origin rpy="0 0 1" xyz="${-pi/2} 0 0"/>
+        </joint> -->
+        <joint name="${prefix}tool_tip_to_${prefix}base_link" type="fixed">
             <parent link= "${prefix}base_link"/>
             <child link= "${prefix}tool_tip"/>
-            <origin rpy="0 0 1" xyz="${-pi/2} 0 0"/>
+            <origin xyz="0 0 ${eef_bottom_distance_from_center+eef_tip_distance_from_center}" rpy="0 0 0" />
         </joint>
     </xacro:macro>

File: kr210_pen_support/urdf/macros/kr210_pen_macro.xacro (robot description, xacro)
@@ -11,9 +11,9 @@
   <xacro:include filename="$(find kr210_pen_support)/urdf/parts/kl2000_console_h400_macro.xacro"/>
   <!-- Kuka KR210R2700extra robot -->
-  <xacro:include filename="$(find kr210_robot_support)/urdf/macros/kr210_macro.xacro"/>
+  <xacro:include filename="$(find kuka_kr210_support)/urdf/kr210r2700extra_macro.xacro"/>
   <!-- Welding Table -->
   <xacro:include filename="$(find kr210_pen_support)/urdf/parts/forster_welding_table_macro.xacro"/>
   <!-- Penholder End Effector -->
-  <xacro:include filename="$(find kr210_pen_support)/urdf/parts/penholder_macro.xacro"/>
+  <xacro:include filename="$(find kr210_eef_support)/urdf/penholder_macro.xacro"/>
   <!-- MACRO START  -->
   <xacro:macro name="kr210_pen" params="prefix">
@@ -21,5 +21,5 @@
     <xacro:kl2000 prefix="${prefix}kl2000_"/>
     <xacro:kl2000_console_h400 prefix="${prefix}console_"/>
-    <xacro:kr210 prefix="${prefix}"/>
+    <xacro:kuka_kr210r2700extra prefix="${prefix}kr210_"/>
     <xacro:forster_welding_table prefix="${prefix}table_"/>
     <xacro:penholder prefix="${prefix}penholder_"/>
@@ -38,5 +38,5 @@
     </joint>
     <!-- Welding table to linear track -->
-    <joint name="${prefix}base_link_to_${prefix}kl2000_mobile_base" type="fixed">
+    <joint name="${prefix}table_base_link_to_${prefix}kl2000_mobile_base" type="fixed">
       <parent link="${prefix}kl2000_base_link"/>
       <child link="${prefix}table_base_link"/>
@@ -44,8 +44,8 @@
     </joint>
     <!-- End effector to robot -->
-    <joint name="${prefix}penholder_eef_base_link_to_${prefix}quick_release_base_link" type="fixed">
-      <parent link="${prefix}kr210_qr_tool0"/>
+    <joint name="${prefix}penholder_base_link_to_${prefix}kr210_tool0" type="fixed">
+      <parent link="${prefix}kr210_tool0"/>
       <child link="${prefix}penholder_base_link"/>
-      <origin xyz="0 0 0.02" rpy="${pi} 0 ${pi*(5/6)}"/>
+      <origin xyz="0 0 0" rpy="0 0 0"/>
     </joint>
   </xacro:macro>

Commit message: Correct name of launchers

File: kr210_eef_support/urdf/penholder_macro.xacro (robot description, xacro)
@@ -4,18 +4,4 @@
   <xacro:property name="eef_tip_distance_from_center" value="0.2294"/>
     <xacro:macro name="penholder" params="prefix">
-        <!--<link name="${prefix}base_link">
-            <visual>
-                <origin xyz="0 0 0" rpy="${pi/2} 0 0"/>
-                <geometry>
-                    <mesh filename="package://kr210_pen_support/meshes/visual/KUKA_Quickrelease_Flange_visual.dae" scale="0.001 0.001 0.001"/>
-                </geometry>
-            </visual>
-            <collision>
-                <origin xyz="0 0 0" rpy="${pi/2} 0 0"/>
-                <geometry>
-                    <mesh filename="package://kr210_pen_support/meshes/collision/KUKA_Quickrelease_Flange_collision.stl" scale="0.001 0.001 0.001"/>
-                </geometry>
-            </collision>
-        </link> -->
         <link name="${prefix}base_link">
             <visual>
@@ -33,9 +19,4 @@
         </link>
         <link name="${prefix}tool_tip"/>
-        <!-- <joint name="${prefix}eef_base_link_to_${prefix}base_link" type="fixed">
-            <parent link= "${prefix}base_link"/>
-            <child link= "${prefix}eef_base_link"/>
-            <origin rpy="0 0 1" xyz="${-pi/2} 0 0"/>
-        </joint> -->
         <joint name="${prefix}tool_tip_to_${prefix}base_link" type="fixed">
             <parent link= "${prefix}base_link"/>
