Commit message: correct tangent vector of the atl ee

File: kr210_eef_support/urdf/atl_tool_macro.xacro (robot description, xacro)
@@ -35,5 +35,5 @@
             <parent link= "${prefix}base_link"/>
             <child link= "${prefix}tool_tip"/>
-            <origin xyz="0 ${eef_tip_y_distance_from_center} ${eef_bottom_distance_from_center+eef_tip_z_distance_from_center}" rpy="0 0 0" />
+            <origin xyz="0 ${eef_tip_y_distance_from_center} ${eef_bottom_distance_from_center+eef_tip_z_distance_from_center}" rpy="0 0 ${-pi}" />
         </joint>
     </xacro:macro>

Commit message: Remove -pi that was rotating the tool axis

File: kr210_eef_support/urdf/atl_tool_macro.xacro (robot description, xacro)
@@ -35,5 +35,5 @@
             <parent link= "${prefix}base_link"/>
             <child link= "${prefix}tool_tip"/>
-            <origin xyz="0 ${eef_tip_y_distance_from_center} ${eef_bottom_distance_from_center+eef_tip_z_distance_from_center}" rpy="0 0 ${-pi}" />
+            <origin xyz="0 ${eef_tip_y_distance_from_center} ${eef_bottom_distance_from_center+eef_tip_z_distance_from_center}" rpy="0 0 0" />
         </joint>
     </xacro:macro>
